Commit message: Summertime

File: real_ws/src/fmauch_universal_robot/ur_description/urdf/inc/ur_macro.xacro (robot description, xacro)
@@ -316,5 +316,4 @@
       <child link="${prefix}tool0"/>
     </joint>
-<!--
     <link name="ground_plane_box">
         <visual>
@@ -337,7 +336,6 @@
         <parent link="world" />
         <child link="ground_plane_box" />
-        <origin xyz="-0.26 0.26 0.69" rpy="0 0 0" />
-    </joint>
--->
+        <origin xyz="-0.3 0 -0.05" rpy="0 0 -0.785" />
+    </joint>
     <link name="world">
     </link>
@@ -345,5 +343,5 @@
         <parent link="world" />
         <child link="base_link"/>
-        <origin xyz="0 0 0.74" rpy="0 0 -0.7854"/>
+        <origin xyz="0 0 0" rpy="0 0 0"/>
     </joint>
     <link name="camera_link">

Commit message: plank

File: real_ws/src/fmauch_universal_robot/ur_description/urdf/inc/ur_macro.xacro (robot description, xacro)
@@ -352,4 +352,26 @@
         <origin xyz="0 0 0" rpy="0 0 0" />
     </joint>
+    <link name="cam_tool">
+        <visual>
+            <origin xyz="0 0 0" rpy="0 0 0"/>
+            <geometry>
+                <box size="1 0.1 0.03"/>
+            </geometry>
+            <material name="Grey">
+                <color rgba="0 1 0 0.05"/>
+            </material>
+        </visual>
+        <collision>
+            <origin xyz="0 0 0" rpy="0 0 0"/>
+            <geometry>
+                <box size="0.1 0.1 0.01"/>
+            </geometry>
+        </collision>
+    </link>
+    <joint name="cam_tool" type="fixed">
+        <parent link="${prefix}tool0" />
+        <child link="cam_tool" />
+        <origin xyz="0 0 0.02" rpy="0 0 0" />
+    </joint>
   </xacro:macro>
 </robot>
